Commit message: feat(arm): M1b 模型对齐 + arm_bringup 只读镜像节点 + 标定限位换算进 URDF
arm_bringup（新包，ament_python）
- real_joint_states：**只读**把真机关节角按 q_urdf = sign·q_ours + zero_shift 发 /joint_states，
  供 robot_state_publisher/RViz 实时镜像真机（模型对齐 + 只读监视）
- 参数默认值取自 arm_description/config/align.yaml（单一真源）⇒ 重启不丢对齐结果
- 安全：绝不 enable()，每轮只发 6 条 0x7FF 刷新帧；连续 max_fail_streak 轮读失败就 FATAL 退出（不装死）
- launch/real_display.launch.py（rsp + rviz2，含 use_rviz/use_gripper/rate_hz）

模型对齐（M1b，详见 docs/TESTING.md §十三）
- 定法：把真机摆成"参考项目初始位姿 + j1 俯视逆时针 90°"（= 模型 (1.5708,0,0,0,0,0)），
  用只读读数一次解出 6 组 (sign, zero_shift)：zero_shift = q_target − sign·q_ours
- 新增 arm_description/config/align.yaml（真源）：j1~j5 sign=−1、j6 sign=+1；
  zero_shift = +1.529724 / −0.191649 / −0.049248 / −0.157540 / +0.048372 / +1.782591
- 限位换算（sign·我们的限位 + zero_shift）写进 urdf/inc/arm_geometry.urdf.xacro：
  j1 [+1.392202,+1.626143] j2 [−2.379924,−0.191649] j3 [−1.891796,−0.049248]
  j4 [−0.157540,+0.938132] j5 [−0.970641,+0.913381] j6 [−1.359002,+4.924184]
  旁证：j1~j5 全部落在上游参考限位内部
- ⚠️ j2/j3 的换算范围不含"参考初始位姿"（q_urdf=0 在范围外 0.19/0.05 rad）
  ⇒ M5/M6 之前要么把臂停在限位内起步、要么重摆一套更宽的限位

修的两个真机坑（AGENTS 陷阱 #28/#29）
- **USB-CAN 设备号会变**（ttyACM0 → ttyACM1）：joint.yaml 的 channel 改 ttyACM1 + 警告注释；
  节点加"连续失败就退出"，避免再次出现"模型冻住却不知道"
- **joint_state_publisher* 会订阅 /joint_states 再回发**：与镜像节点同时开会打架（模型发抖、两个 rsp）
  ⇒ 文档写明镜像前先确认 Publisher count = 1

文档：AGENTS（§2 三个新包 / §4 真源表 / §5 模型坐标限位 / 陷阱 #27~#29）、TESTING §十三、
      readme（状态表 / 目录树 / 路线进度）；rviz/display.rviz 是 RViz 保存后的补全版（内容仍是 Grid+RobotModel+TF）

验证：colcon build → 4 packages；xacro 展开 + urdfdom 解析通过且限位为换算值；
     进程内假驱动测试全绿（默认值 = align.yaml、换算逻辑、缺回包不编造、连续失败退出、channel 生效）

File: src/arm_description/urdf/arm.urdf.xacro (robot description, xacro)
@@ -3,7 +3,9 @@
   展开：xacro arm.urdf.xacro use_gripper:=false > arm.urdf
   看模型：ros2 launch arm_description display.launch.py
-  ⚠️ joint limit 的 lower/upper 目前是**模型坐标**下的参考值（见 inc/arm_geometry.urdf.xacro
-     顶部注释）：本项目自己标定的零位/软限位与模型零位不是同一姿态，需要 M1b 定出
-     每关节的零点差 δ 与符号 s 后，才能把 src/motor_driver/config/joint.yaml 的值换算进来。
+  ✅ joint limit 已是**本项目标定限位换算到模型坐标**的结果（2026-10-04 M1b 真机实测）：
+     q_urdf = sign * q_ours + zero_shift，sign/zero_shift 见 config/align.yaml；
+     换算公式与结果见 inc/arm_geometry.urdf.xacro 顶部注释。
+     注意我们的标定限位比上游窄很多（j1 只有 ±0.1 rad 左右），且 j2/j3 的换算范围**不含**
+     "参考初始位姿"——真正跑 MoveIt 前要么把臂停在限位内起步，要么重新摆一套更宽的限位。
 -->
 <robot xmlns:xacro="http://www.ros.org/wiki/xacro" name="dm_armx">

File: src/arm_description/urdf/inc/arm_geometry.urdf.xacro (robot description, xacro)
@@ -3,6 +3,14 @@
      （CERN-OHL-W-2.0，见 ../LICENSE-CERN-OHL-W-2.0）。改动：mesh 包路径重写；
      夹爪 link/joint 移到 gripper.urdf.xacro；effort/velocity 换成本项目电机实测值；
-     fixed joint 去掉 axis。⚠️ joint limit 的 lower/upper 仍是**模型坐标**下的参考值，
-     待 M1b 用 src/motor_driver/config/joint.yaml 的标定值换算后替换。 -->
+     fixed joint 去掉 axis；**joint limit 换成本项目标定值**（见下）。
+     joint limit 换算（2026-10-04 M1b 真机实测）：
+         q_urdf = sign * q_ours + zero_shift        （sign/zero_shift 见 ../config/align.yaml）
+         lower/upper = sign * (joint.yaml 的 position_min/max) + zero_shift，再按小/大排序
+     真源：src/motor_driver/config/joint.yaml（本项目标定限位） + config/align.yaml（模型对齐）
+     换算结果（模型坐标）：
+         joint1 [+1.392202, +1.626143]    joint2 [-2.379924, -0.191649]
+         joint3 [-1.891796, -0.049248]    joint4 [-0.157540, +0.938132]
+         joint5 [-0.970641, +0.913381]    joint6 [-1.359002, +4.924184]（整圈 ±180°，宽 2π）
+     旁证：j1~j5 换算后全部落在上游参考限位内部。 -->
 <robot name="dm_armx">
   <material name="gripper_finger_black">
@@ -330,5 +338,5 @@
     <child link="link1" />
     <axis xyz="0 0 1" />
-    <limit lower="-2.8" upper="2.8" effort="12" velocity="10" />
+    <limit lower="1.392202" upper="1.626143" effort="12" velocity="10" />
   </joint>
   <joint name="joint2" type="revolute">
@@ -337,5 +345,5 @@
     <child link="link2" />
     <axis xyz="0 0 -1" />
-    <limit lower="-3.14" upper="0" effort="12" velocity="10" />
+    <limit lower="-2.379924" upper="-0.191649" effort="12" velocity="10" />
   </joint>
   <joint name="joint3" type="revolute">
@@ -344,5 +352,5 @@
     <child link="link3" />
     <axis xyz="0 0 1" />
-    <limit lower="-3.14" upper="0" effort="12" velocity="10" />
+    <limit lower="-1.891796" upper="-0.049248" effort="12" velocity="10" />
   </joint>
   <joint name="joint4" type="revolute">
@@ -351,5 +359,5 @@
     <child link="link4" />
     <axis xyz="0 0 1" />
-    <limit lower="-1.87" upper="1.57" effort="3.5" velocity="30" />
+    <limit lower="-0.157540" upper="0.938132" effort="3.5" velocity="30" />
   </joint>
   <joint name="joint5" type="revolute">
@@ -358,5 +366,5 @@
     <child link="link5" />
     <axis xyz="0 0 1" />
-    <limit lower="-1.57" upper="1.57" effort="3.5" velocity="30" />
+    <limit lower="-0.970641" upper="0.913381" effort="3.5" velocity="30" />
   </joint>
   <joint name="joint6" type="revolute">
@@ -365,5 +373,5 @@
     <child link="link6" />
     <axis xyz="0 0 1" />
-    <limit lower="-3.14" upper="3.14" effort="3.5" velocity="30" />
+    <limit lower="-1.359002" upper="4.924184" effort="3.5" velocity="30" />
   </joint>
   <joint name="end_joint" type="fixed">

Commit message: feat(m2): mock 链路跑通（controller_manager + JTC + 广播器）；放宽 j2/j3 限位
M2（**全程未接真机**）
- arm_bringup/config/ros2_controllers.yaml：update_rate 100；joint_state_broadcaster +
  arm_controller（joint_trajectory_controller，6 关节；命令 position / 状态 position+velocity）
- arm_bringup/launch/mock_control.launch.py：ros2_control_node（mock_components/GenericSystem）
  + robot_state_publisher + spawner(jsb) → spawner(arm_controller) + rviz2
- arm_bringup/setup.py：data_files 改用 glob('launch/*.py') + glob('config/*.yaml')
- arm_description 的 mock initial_value 由 0 改成限位内的 (1.51,-1.0,-0.9,0.3,0,0)（FK 验证不自交）

验收证据：
- ros2 control list_controllers → 两个都 active；list_hardware_interfaces → 6 个 position 命令接口 claimed
- 发两点轨迹（终点 (1.45,-1.10,-0.80,0.35,0.10,0.10)）→ "Goal successfully reached!"
  且 /joint_states 的 position 精确变成该终点值

限位放宽（用户决定，2026-10-04）
- joint.yaml 的 j2/j3 position_min：0.0 → −0.25 / −0.10
- 理由：真机"自然停放姿态"是 q_ours = −0.1916 / −0.0477，原限位不含它 ⇒
  第一个"保持当前位置"就会被钳成 11° / 2.7° 的运动（陷阱 #21 的翻版）
- 换算后的 URDF 限位 → j2 [−2.379924, +0.058351]、j3 [−1.891796, +0.050752]
- ⚠️ 代价：q_urdf = 0 离 j2 上界只剩 0.058 rad（3.3°）

文档：AGENTS §5（模型坐标限位 + 放宽说明）、TESTING §十三（放宽记录 + M2 验收）、arm_description/README

File: src/arm_description/urdf/arm.urdf.xacro (robot description, xacro)
@@ -6,6 +6,6 @@
      q_urdf = sign * q_ours + zero_shift，sign/zero_shift 见 config/align.yaml；
      换算公式与结果见 inc/arm_geometry.urdf.xacro 顶部注释。
-     注意我们的标定限位比上游窄很多（j1 只有 ±0.1 rad 左右），且 j2/j3 的换算范围**不含**
-     "参考初始位姿"——真正跑 MoveIt 前要么把臂停在限位内起步，要么重新摆一套更宽的限位。
+     注意我们的标定限位比上游窄很多（j1 只有 ±0.1 rad 左右）；j2/j3 的下界当天放宽过
+     （让"自然停放姿态"落进限位内，见 inc/arm_geometry.urdf.xacro 顶部注释）。
 -->
 <robot xmlns:xacro="http://www.ros.org/wiki/xacro" name="dm_armx">

File: src/arm_description/urdf/inc/arm.ros2_control.xacro (robot description, xacro)
@@ -5,5 +5,8 @@
      M5 接真机时只换 <plugin>（motor_driver_hardware/DmSystemInterface）并补关节参数
      （motor_id / motor_type / offset / direction / limit / torque_max，真源仍是
-      src/motor_driver/config/joint.yaml）。 -->
+      src/motor_driver/config/joint.yaml）。
+     ⚠️ 每个关节的 `initial_value` 是 **mock 的起始姿态**，必须落在**换算后的限位**里
+     （限位见 arm_geometry.urdf.xacro 顶部）：这里取 (1.51, -1.0, -0.9, 0.3, 0.0, 0.0)，
+     FK 验证不自交（非相邻连杆最小间距 4.9 cm）。**写 0 会落在 j1~j3 换算后的限位之外**。 -->
 <robot xmlns:xacro="http://www.ros.org/wiki/xacro">
   <xacro:macro name="arm_ros2_control" params="name:=ArmMockSystem">
@@ -14,20 +17,20 @@
       <joint name="joint1">
         <command_interface name="position"/>
-        <state_interface name="position"><param name="initial_value">0.0</param></state_interface>
+        <state_interface name="position"><param name="initial_value">1.51</param></state_interface>
         <state_interface name="velocity"/>
       </joint>
       <joint name="joint2">
         <command_interface name="position"/>
-        <state_interface name="position"><param name="initial_value">0.0</param></state_interface>
+        <state_interface name="position"><param name="initial_value">-1.0</param></state_interface>
         <state_interface name="velocity"/>
       </joint>
       <joint name="joint3">
         <command_interface name="position"/>
-        <state_interface name="position"><param name="initial_value">0.0</param></state_interface>
+        <state_interface name="position"><param name="initial_value">-0.9</param></state_interface>
         <state_interface name="velocity"/>
       </joint>
       <joint name="joint4">
         <command_interface name="position"/>
-        <state_interface name="position"><param name="initial_value">0.0</param></state_interface>
+        <state_interface name="position"><param name="initial_value">0.3</param></state_interface>
         <state_interface name="velocity"/>
       </joint>

File: src/arm_description/urdf/inc/arm_geometry.urdf.xacro (robot description, xacro)
@@ -9,7 +9,9 @@
      真源：src/motor_driver/config/joint.yaml（本项目标定限位） + config/align.yaml（模型对齐）
      换算结果（模型坐标）：
-         joint1 [+1.392202, +1.626143]    joint2 [-2.379924, -0.191649]
-         joint3 [-1.891796, -0.049248]    joint4 [-0.157540, +0.938132]
+         joint1 [+1.392202, +1.626143]    joint2 [-2.379924, +0.058351]
+         joint3 [-1.891796, +0.050752]    joint4 [-0.157540, +0.938132]
          joint5 [-0.970641, +0.913381]    joint6 [-1.359002, +4.924184]（整圈 ±180°，宽 2π）
+     2026-10-04 放宽 j2/j3 下界（joint.yaml：0.0 → −0.25 / −0.10）：真机"自然停放姿态"在
+     q_ours = −0.1916 / −0.0477，原限位不含它 ⇒ 第一个"保持当前位置"会被钳成一次 11° / 2.7° 的运动。
      旁证：j1~j5 换算后全部落在上游参考限位内部。 -->
 <robot name="dm_armx">
@@ -345,5 +347,5 @@
     <child link="link2" />
     <axis xyz="0 0 -1" />
-    <limit lower="-2.379924" upper="-0.191649" effort="12" velocity="10" />
+    <limit lower="-2.379924" upper="0.058351" effort="12" velocity="10" />
   </joint>
   <joint name="joint3" type="revolute">
@@ -352,5 +354,5 @@
     <child link="link3" />
     <axis xyz="0 0 1" />
-    <limit lower="-1.891796" upper="-0.049248" effort="12" velocity="10" />
+    <limit lower="-1.891796" upper="0.050752" effort="12" velocity="10" />
   </joint>
   <joint name="joint4" type="revolute">
