Commit message: feat(desc): 夹爪质量/质心做成可切换的一路（默认仍走空载辨识版）
背景：实物 joint6 是**空载**（只有 link6 本体），URDF 模型比实机多一截
（end_link + gripper_tcp），后续要跟夹爪一起加回来。

- apply_identified_inertia.py 加 --gripper：
  * 不带（默认）：end_link + gripper_tcp 惯量清零 —— 与原先一致，产出**空载**辨识版
  * 带 --gripper：只清 gripper_tcp，end_link（夹爪底座）保留自己的惯量，
    并注入 gravity_identified.yaml 新增的 gripper: 段（各 link 质量/质心）
- gravity_identified.yaml 加 gripper_meta: + gripper: 两段；link6 的辨识值**不动**
  （0.7718 kg 是空载辨识值 —— 它已经是量空载的，别再"减掉 joint6 负载"，
   那样会把 j2/j4 前馈弄错约 0.8 N·m）
- gripper.urdf.xacro 的指节 link 给零 <inertial>（质量真源统一在 yaml，避免两处漂）
- CMake 加第三份 URDF arm_identified_gripper.urdf 与中间产物 arm_dynamics_gripper.urdf

⚠️ 夹爪那几个质量/质心是**上游 CAD 名义值的占位**，没辨识过；真装上夹爪后必须重辨。

File: src/arm_description/urdf/inc/gripper.urdf.xacro (robot description, xacro)
@@ -1,7 +1,16 @@
 <?xml version="1.0"?>
-<!-- 夹爪几何（finger_left/right，prismatic）。默认不加载：主文件用 use_gripper 参数控制。 -->
+<!-- 夹爪几何（finger_left/right，prismatic）。默认不加载：主文件用 use_gripper 参数控制。
+  ⚠️ 两个手指的 inertial 故意留**零**：真源是 config/gravity_identified.yaml 的 `gripper:` 段，
+     由 scripts/apply_identified_inertia.py（带 gripper 开关）注入 —— 夹爪没辨识过，那里的数是占位。
+     这里写零是为了让 `use_gripper:=true` 的**几何/显示**与**动力学**只有一个质量真源。 -->
 <robot name="dm_armx_gripper" xmlns:xacro="http://www.ros.org/wiki/xacro">
   <xacro:macro name="gripper_links">
     <link name="finger_left_link">
+      <!-- 质量真源见文件头注释（脚本带 gripper 开关时注入） -->
+      <inertial>
+        <origin xyz="0 0 0" rpy="0 0 0" />
+        <mass value="0.0" />
+        <inertia ixx="0.0" ixy="0.0" ixz="0.0" iyy="0.0" iyz="0.0" izz="0.0" />
+      </inertial>
       <visual name="finger_left_body">
         <origin xyz="0 0 0" rpy="0 0 0" />
@@ -40,4 +49,10 @@
     </link>
     <link name="finger_right_link">
+      <!-- 质量真源见文件头注释（脚本带 gripper 开关时注入） -->
+      <inertial>
+        <origin xyz="0 0 0" rpy="0 0 0" />
+        <mass value="0.0" />
+        <inertia ixx="0.0" ixy="0.0" ixz="0.0" iyy="0.0" iyz="0.0" izz="0.0" />
+      </inertial>
       <visual name="finger_right_body">
         <origin xyz="0 0 0" rpy="0 0 0" />
