Commit message: feat(m5): ros2_control 硬件接口插件 DmSystemInterface（接真机，默认只读）
插件（motor_driver_hardware，新增 dm_system_interface.{hpp,cpp} + pluginlib xml）
- 参数**全部来自 <param>**：device/baud/enable_on_activate/vlim + 每关节
  motor_id/motor_type/direction/offset/p_max/v_max/t_max/position_min/position_max/
  **sign/zero_shift**（模型对齐）/可选 PID
- 三层坐标：模型坐标 --sign/δ--> q_ours --direction/offset--> 电机 p_m；
  换算函数只有一份（dm_joint.hpp 的 model_to_ours/ours_to_model，插件与测试共用）
- 生命周期：on_init 解析校验 → on_configure 建串口/总线/关节 →
  on_activate 开串口 + sync_states + 写 0x0A=2（+可选 PID）+ 可选使能 → on_deactivate **全部失能**
- read()：poll + 填 position/velocity（模型坐标）+ **ERR 非 0/1 报 ERROR**（让 CM 停控制器）
- write()：**命令是 NaN 就发保持帧**（用电机侧实测位置，绝不当 0）；`enable_on_activate=false` 时
  **一个控制帧都不发**（只发 0x7FF 刷新帧读状态）
- 用新版 on_init(HardwareComponentInterfaceParams) 签名（老的已 deprecated，构建零警告）

xacro（arm_description/urdf/inc/arm.ros2_control.xacro）
- 加 `use_mock` 开关（默认 true，M2 的 mock 链路保留）
- 真机分支：**xacro 直接读 motor_driver/config/joint.yaml（设备/档位/限位/direction/offset）
  + arm_description/config/align.yaml（sign/δ）生成 <param>** ⇒ 单一真源不破

launch（arm_bringup/launch/real_control.launch.py，新增）
- 默认 `enable_on_activate=false` + 只起状态广播器 = **只读**（最安全的一步）
- 三步验收：只读 → `enable_on_activate:=true`（保持）→ 再加 `spawn_arm_controller:=true vlim:=0.5`

测试（假串口 + 模拟电机，5 用例；全仓库 27 用例）
- 只读模式一个控制帧都不发；激活时先写 0x0A=2 再使能再补保持帧（保持帧用电机侧实测值）；
  命令 NaN 继续保持；**模型坐标 0 ⇒ 电机侧 1.785878**（M1b 实测解出来的数，闭环读回一致）；
  ERR=0x0D ⇒ read() 报 ERROR 且 deactivate 全失能；参数错误在 on_init/on_configure 就拒
- 验收：colcon test --packages-select motor_driver_hardware → 27 tests, 0 errors, 0 failures

两个环境/API 坑（AGENTS 陷阱 #32/#33）
- 链接 rclcpp 的**可执行文件**报「找不到 -lcap / -llttng-ust」：库在 $CONDA_PREFIX/lib 但 pixi
  激活不设 LIBRARY_PATH ⇒ CMake 里 link_directories($ENV{CONDA_PREFIX}/lib)
- hardware_interface 的 on_init(HardwareInfo&) 在 jazzy 已 deprecated ⇒ 换新签名

文档：AGENTS（§1 现状、§2 该行、§3 插件 API、§5 三层坐标、§6 #32/#33、§7 插件测试法）、
readme（状态表 / 路线 / 三步验收）、TESTING（M5 记录 + 两个测试自己的错）、包内 README（五层 + 三步验收）

File: src/arm_description/urdf/inc/arm.ros2_control.xacro (robot description, xacro)
@@ -1,48 +1,84 @@
 <?xml version="1.0"?>
-<!-- ros2_control 硬件接口。
-     现在（M1/M2）用 ros2_control 自带的 mock：不接真机也能把
-     controller_manager → joint_trajectory_controller → joint_state_broadcaster 跑通。
-     M5 接真机时只换 <plugin>（motor_driver_hardware/DmSystemInterface）并补关节参数
-     （motor_id / motor_type / offset / direction / limit / torque_max，真源仍是
-      src/motor_driver/config/joint.yaml）。
-     ⚠️ 每个关节的 `initial_value` 是 **mock 的起始姿态**，必须落在**换算后的限位**里
-     （限位见 arm_geometry.urdf.xacro 顶部）：这里取 (1.51, -1.0, -0.9, 0.3, 0.0, 0.0)，
-     FK 验证不自交（非相邻连杆最小间距 4.9 cm）。**写 0 会落在 j1~j3 换算后的限位之外**。 -->
+<!-- ros2_control 硬件接口。两条分支由 `use_mock` 选：
+     - `use_mock:=true`（默认）：ros2_control 自带的 mock —— 不接真机就能把
+       controller_manager → joint_trajectory_controller → joint_state_broadcaster 跑通（M2 的验收链路）。
+     - `use_mock:=false`：真插件 `motor_driver_hardware/DmSystemInterface`。关节参数**由 xacro 直接从**
+       - `motor_driver/config/joint.yaml`（direction / offset / 档位 / 软限位 / 串口设备）
+       - `arm_description/config/align.yaml`（模型对齐 sign / zero_shift）
+       **读出来**生成 <param> ⇒ 单一真源不破，不用在两处维护同一批数字。
+     ⚠️ mock 分支的 `initial_value` 是**起始姿态**，必须落在换算后的限位里（见 arm_geometry.urdf.xacro 顶部）：
+        取 (1.51, -1.0, -0.9, 0.3, 0.0, 0.0)，FK 验证不自交。写 0 会落在 j1~j3 换算后的限位之外。
+     ⚠️ 真机分支默认 `enable_on_activate:=false`：**只读**（不使能、不发控制帧），
+        首轮验收先这么跑；要动电机必须显式传 true。 -->
 <robot xmlns:xacro="http://www.ros.org/wiki/xacro">
-  <xacro:macro name="arm_ros2_control" params="name:=ArmMockSystem">
+  <xacro:arg name="use_mock" default="true"/>
+  <xacro:arg name="enable_on_activate" default="false"/>
+  <xacro:arg name="vlim" default="1.0"/>
+  <xacro:arg name="joint_cfg" default="$(find motor_driver)/config/joint.yaml"/>
+  <xacro:arg name="align_cfg" default="$(find arm_description)/config/align.yaml"/>
+  <xacro:property name="arm_cfg" value="${xacro.load_yaml('$(arg joint_cfg)')}"/>
+  <xacro:property name="align_cfg" value="${xacro.load_yaml('$(arg align_cfg)')}"/>
+  <!-- mock 的一个关节：起始姿态用 initial（模型坐标） -->
+  <xacro:macro name="mock_joint" params="name initial">
+    <joint name="${name}">
+      <command_interface name="position"/>
+      <state_interface name="position"><param name="initial_value">${initial}</param></state_interface>
+      <state_interface name="velocity"/>
+    </joint>
+  </xacro:macro>
+  <!-- 真机的一个关节：参数全部从上面两个 yaml 里取 -->
+  <xacro:macro name="real_joint" params="name">
+    <xacro:property name="jcfg" value="${arm_cfg['joints'][name]}"/>
+    <xacro:property name="acfg" value="${align_cfg['joints'][name]}"/>
+    <joint name="${name}">
+      <command_interface name="position"/>
+      <state_interface name="position"/>     <!-- 真值从硬件读，不给 initial_value -->
+      <state_interface name="velocity"/>
+      <param name="motor_id">${jcfg['slave_id']}</param>
+      <param name="motor_type">${jcfg['motor_type']}</param>
+      <param name="direction">${jcfg['direction']}</param>
+      <param name="offset">${jcfg['offset']}</param>
+      <param name="p_max">${jcfg['limit'][0]}</param>
+      <param name="v_max">${jcfg['limit'][1]}</param>
+      <param name="t_max">${jcfg['limit'][2]}</param>
+      <param name="position_min">${jcfg['position_min']}</param>
+      <param name="position_max">${jcfg['position_max']}</param>
+      <!-- 模型对齐：q_urdf = sign · q_ours + zero_shift -->
+      <param name="sign">${acfg['sign']}</param>
+      <param name="zero_shift">${acfg['zero_shift']}</param>
+    </joint>
+  </xacro:macro>
+  <xacro:macro name="arm_ros2_control" params="name:=ArmSystem">
     <ros2_control name="${name}" type="system">
-      <hardware>
-        <plugin>mock_components/GenericSystem</plugin>
-      </hardware>
-      <joint name="joint1">
-        <command_interface name="position"/>
-        <state_interface name="position"><param name="initial_value">1.51</param></state_interface>
-        <state_interface name="velocity"/>
-      </joint>
-      <joint name="joint2">
-        <command_interface name="position"/>
-        <state_interface name="position"><param name="initial_value">-1.0</param></state_interface>
-        <state_interface name="velocity"/>
-      </joint>
-      <joint name="joint3">
-        <command_interface name="position"/>
-        <state_interface name="position"><param name="initial_value">-0.9</param></state_interface>
-        <state_interface name="velocity"/>
-      </joint>
-      <joint name="joint4">
-        <command_interface name="position"/>
-        <state_interface name="position"><param name="initial_value">0.3</param></state_interface>
-        <state_interface name="velocity"/>
-      </joint>
-      <joint name="joint5">
-        <command_interface name="position"/>
-        <state_interface name="position"><param name="initial_value">0.0</param></state_interface>
-        <state_interface name="velocity"/>
-      </joint>
-      <joint name="joint6">
-        <command_interface name="position"/>
-        <state_interface name="position"><param name="initial_value">0.0</param></state_interface>
-        <state_interface name="velocity"/>
-      </joint>
+      <xacro:if value="$(arg use_mock)">
+        <hardware>
+          <plugin>mock_components/GenericSystem</plugin>
+        </hardware>
+      </xacro:if>
+      <xacro:unless value="$(arg use_mock)">
+        <hardware>
+          <plugin>motor_driver_hardware/DmSystemInterface</plugin>
+          <param name="device">${arm_cfg['channel']}</param>
+          <param name="baud">${arm_cfg['baud']}</param>
+          <param name="enable_on_activate">$(arg enable_on_activate)</param>
+          <param name="vlim">$(arg vlim)</param>
+        </hardware>
+      </xacro:unless>
+      <xacro:if value="$(arg use_mock)">
+        <xacro:mock_joint name="joint1" initial="1.51"/>
+        <xacro:mock_joint name="joint2" initial="-1.0"/>
+        <xacro:mock_joint name="joint3" initial="-0.9"/>
+        <xacro:mock_joint name="joint4" initial="0.3"/>
+        <xacro:mock_joint name="joint5" initial="0.0"/>
+        <xacro:mock_joint name="joint6" initial="0.0"/>
+      </xacro:if>
+      <xacro:unless value="$(arg use_mock)">
+        <xacro:real_joint name="joint1"/>
+        <xacro:real_joint name="joint2"/>
+        <xacro:real_joint name="joint3"/>
+        <xacro:real_joint name="joint4"/>
+        <xacro:real_joint name="joint5"/>
+        <xacro:real_joint name="joint6"/>
+      </xacro:unless>
     </ros2_control>
   </xacro:macro>

Commit message: feat(m5): 2.4.2 MIT 参数解析（**行为不变**，一个字都还没用上）
- 新增 arm_description/config/mit_gains.yaml：每关节 kp_hold / kd_hold。
  **不塞进 motor_driver/config/joint.yaml** —— 那份是 Python 驱动层的真源，arm_config.py
  用 dataclass 严格解析（多一个键就 TypeError），塞进去会连带改 Python 包；而 kp/kd 只是
  ros2_control 侧的控制器增益，与驱动层无关。
  ⚠️ 值（7.0 / 0.8）是 **DESIGN 的占位参考值，不是标定结果**：§D5b 说 4340P 与 4310 的 kp
  量级差 5 倍以上，2.4.4 要逐关节标定。
- arm.ros2_control.xacro：加 <xacro:arg name="gravity_ff" default="false"/>；真机分支从
  joint.yaml 取 torque_max（12.0/3.5，**关节侧额定值**，与档位里的 t_max=电机峰值 28/10
  不是一回事）、从 mit_gains.yaml 取 kp_hold/kd_hold，连同 urdf_path 一起变成 <param>。
- DmSystemInterface：解析 gravity_ff / urdf_path（存成员）与每关节 torque_max（进
  cfg.torque_max）/ kp_hold / kd_hold（进 JointParams）。**全部尚未使用**：mode 仍写死 2、
  on_activate 仍写 0x0A=2、write() 仍只走 set_pos_vel。
  仅当 gravity_ff=true 时才校验这些参数（默认 false 不该拦住任何东西）。
- 启动日志多打 gravity_ff / urdf_path，每关节多打 tm/kp/kd。

验证：单元测试 34/0；真机只读链路 0 错误，日志确认 6 关节 tm12.0/3.5、kp7.0、kd0.8、
gravity_ff=false、urdf_path 指向构建时生成的那份 URDF。

File: src/arm_description/urdf/inc/arm.ros2_control.xacro (robot description, xacro)
@@ -4,6 +4,7 @@
        controller_manager → joint_trajectory_controller → joint_state_broadcaster 跑通（M2 的验收链路）。
      - `use_mock:=false`：真插件 `motor_driver_hardware/DmSystemInterface`。关节参数**由 xacro 直接从**
-       - `motor_driver/config/joint.yaml`（direction / offset / 档位 / 软限位 / 串口设备）
+       - `motor_driver/config/joint.yaml`（direction / offset / 档位 / 软限位 / torque_max / 串口设备）
        - `arm_description/config/align.yaml`（模型对齐 sign / zero_shift）
+       - `arm_description/config/mit_gains.yaml`（MIT 保持增益 kp_hold / kd_hold）
        **读出来**生成 <param> ⇒ 单一真源不破，不用在两处维护同一批数字。
      ⚠️ mock 分支的 `initial_value` 是**起始姿态**，必须落在换算后的限位里（见 arm_geometry.urdf.xacro 顶部）：
@@ -15,8 +16,13 @@
   <xacro:arg name="enable_on_activate" default="false"/>
   <xacro:arg name="vlim" default="1.0"/>
+  <!-- 重力前馈总开关：true ⇒ 这条链的关节进 MIT（每关节 0x0A=1）+ 力矩前馈。
+       默认 false ⇒ 一切照旧走 POS_VEL。2.4.2 只把它传进 <param>，插件还不用。 -->
+  <xacro:arg name="gravity_ff" default="false"/>
   <xacro:arg name="joint_cfg" default="$(find motor_driver)/config/joint.yaml"/>
   <xacro:arg name="align_cfg" default="$(find arm_description)/config/align.yaml"/>
+  <xacro:arg name="mit_gains_cfg" default="$(find arm_description)/config/mit_gains.yaml"/>
   <xacro:property name="arm_cfg" value="${xacro.load_yaml('$(arg joint_cfg)')}"/>
   <xacro:property name="align_cfg" value="${xacro.load_yaml('$(arg align_cfg)')}"/>
+  <xacro:property name="mit_cfg" value="${xacro.load_yaml('$(arg mit_gains_cfg)')}"/>
   <!-- mock 的一个关节：起始姿态用 initial（模型坐标） -->
   <xacro:macro name="mock_joint" params="name initial">
@@ -30,8 +36,9 @@
     </joint>
   </xacro:macro>
-  <!-- 真机的一个关节：参数全部从上面两个 yaml 里取 -->
+  <!-- 真机的一个关节：参数全部从上面三个 yaml 里取 -->
   <xacro:macro name="real_joint" params="name">
     <xacro:property name="jcfg" value="${arm_cfg['joints'][name]}"/>
     <xacro:property name="acfg" value="${align_cfg['joints'][name]}"/>
+    <xacro:property name="mcfg" value="${mit_cfg['joints'][name]}"/>
     <joint name="${name}">
       <command_interface name="position"/>
@@ -53,4 +60,10 @@
       <param name="sign">${acfg['sign']}</param>
       <param name="zero_shift">${acfg['zero_shift']}</param>
+      <!-- MIT（gravity_ff:=true）才用得上：力矩上限 + 保持增益。
+           torque_max 是**关节侧额定值**（j1~j3 12.0 / j4~j6 3.5），与上面档位里的
+           t_max（电机峰值 28/10）不是一回事。2.4.2 只解析，不使用。 -->
+      <param name="torque_max">${jcfg['torque_max']}</param>
+      <param name="kp_hold">${mcfg['kp_hold']}</param>
+      <param name="kd_hold">${mcfg['kd_hold']}</param>
     </joint>
   </xacro:macro>
@@ -72,4 +85,6 @@
                惯性与运动学和运行期那份同源。插件目前**不读**它（2.2/2.4 才接上）。 -->
           <param name="urdf_path">$(find arm_description)/urdf/arm.urdf</param>
+          <!-- 重力前馈总开关。2.4.2 只解析，不使用 ⇒ 现在传 true 也没有任何行为变化。 -->
+          <param name="gravity_ff">$(arg gravity_ff)</param>
         </hardware>
       </xacro:unless>

Commit message: refactor: 砍掉整个 MIT 路径 —— C++ 侧只走 POS_VEL
决定依据（2026-10-14 只读实测，未使能、未写寄存器）：折叠位**失能 5 s 零漂移**
（六台全部 0.000000 rad），torque 全在 ±0.02 N·m（12 位量化噪声）内
⇒ 折叠位的重力由**机械结构**承载，电机没出那个力 ⇒ MIT 的重力前馈在日常姿态上是空转。
本链不需要关节力矩。

C++ 侧改动（Python motor_driver 与 third_party **一律不动**）
- `dm_joint`：只做 POS_VEL。删 `set_mit` / `clamp_mit_torque` /
  `prepare_frame_raw` / `mode()` / `torque_max`（`JointConfig.mode` 字段也已删）
- `dm_system_interface`：控制模式**固定** `0x0A=2`，删掉运行期模式切换状态机与
  `dm_frame_plan` 依赖。`effort` 命令接口**保留为空插槽**（本层永不读），
  这样将来若要加力矩控制器不必改 URDF/xacro
- 删 `dm_frame_plan.hpp`（只有一种模式 ⇒ 无决策可言）+ 其测试 `test_frame_plan.cpp`
- ⚠️ **保留** `dm_frames::mit_frame` / `float_to_uint` 及 `test_dm_frames` 里与 Python 的
  逐字节对拍：那是**协议**层，Python 侧 `joint.py` 仍支持 MIT，两份实现必须继续咬住

控制层与配置
- 删整包 `src/arm_controllers`（`GravityModel` + `GravityFfLaw`，R2 的产品）——
  重力前馈是 MIT 专属，POS_VEL 下固件积分自己抗重力，它没有消费者
- 删 `arm_description/config/mit_gains.yaml`（随之 `arm_description/CMakeLists.txt`
  不再传 `mit_gains_cfg`）、`arm_bringup/config/ros2_controllers_mit.yaml`
- xacro：删 `gravity_ff` 实参、`torque_max`/`kp_hold`/`kd_hold` 参数、
  `velocity` **命令**接口（无控制器声索它；但**保留** position/effort 命令接口，
  且 mock 与真机分支接口集保持一致）
- launch：删 `gravity_ff`/`mit_controllers` 两个参数；控制器配置只剩一份
- 插件描述 / 控制器配置注释同步

测试：39 → 39（净持平，换了内容）。`test_dm_joint` 删 MIT 对拍用例、
`test_iface_wiring` 由 6 条改 4 条（新覆盖"一个 MIT 帧都不该有"）。
`test_dm_joint` 的 POS_VEL 与 Python 对拍、`test_dm_frames` 的 MIT 帧对拍**都保留**。

验证：干净重建（删 build/install/log）9 包通过；
motor_driver_hardware 26 / arm_motion 9 / arm_msgs 4 = 39 tests 全绿。
xacro 展开核对：真机 hw params 只剩 device/baud/enable_on_activate/vlim，
命令接口 `[effort, position]`、状态接口 `[effort, position, velocity]`，mock 与真机一致。
`ros2 launch --show-args` 已无 mit/gravity 参数。
⚠️ 既有失败（与本次无关）：`arm_bringup` "Ran 0 tests / NO TESTS RAN"（该包没有 test/ 目录，
pytest 空跑返回码 5）；另有 arm_application 的 uncrustify 与 motor_driver 的 pytest 环境错。

备查：被砍的 R1+R2 完整实现在分支 `refactor/layers-r1-r2`（commit 8840e26）。

File: src/arm_description/urdf/inc/arm.ros2_control.xacro (robot description, xacro)
@@ -4,8 +4,11 @@
        controller_manager → joint_trajectory_controller → joint_state_broadcaster 跑通（M2 的验收链路）。
      - `use_mock:=false`：真插件 `motor_driver_hardware/DmSystemInterface`。关节参数**由 xacro 直接从**
-       - `motor_driver/config/joint.yaml`（direction / offset / 档位 / 软限位 / torque_max / 串口设备）
+       - `motor_driver/config/joint.yaml`（direction / offset / 档位 / 软限位 / 串口设备）
        - `arm_description/config/align.yaml`（模型对齐 sign / zero_shift）
-       - `arm_description/config/mit_gains.yaml`（MIT 保持增益 kp_hold / kd_hold）
        **读出来**生成 <param> ⇒ 单一真源不破，不用在两处维护同一批数字。
+     ⚠️ **控制模式固定 POS_VEL（`0x0A = 2`）**，MIT 已砍（2026-10-14）：本链不需要关节力矩，
+        而折叠位的重力由机械结构承载（实测：失能 5 s 零漂移）。`effort` 命令接口保留为**空插槽**
+        （本层不读），将来若要加力矩控制器不必改本文件。
+        ⇒ `mit_gains.yaml`（kp_hold/kd_hold/ki_hold/friction_*）与 `torque_max` **不再进 <param>**。
      ⚠️ mock 分支的 `initial_value` 是**起始姿态**，必须落在换算后的限位里（见 arm_geometry.urdf.xacro 顶部）：
         取 (1.51, -1.0, -0.9, 0.3, 0.0, 0.0)，FK 验证不自交。写 0 会落在 j1~j3 换算后的限位之外。
@@ -16,25 +19,14 @@
   <xacro:arg name="enable_on_activate" default="false"/>
   <xacro:arg name="vlim" default="1.0"/>
-  <!-- 预置控制模式（LAYERS §4 的 D-L1）：真实的模式由 **effort 命令接口的 NaN 语义**决定 ——
-       NaN（没有控制器声索力矩）⇒ POS_VEL；有限值（有控制器在写力矩）⇒ MIT。
-       `gravity_ff` 只决定"**还没有控制器时**预置哪一种"：
-         false（默认）⇒ 预置 POS_VEL（固件位置环托住，最稳）
-         true          ⇒ 预置 MIT + `effort`=0（硬件出自己的 PD，**不自算重力**——控制律在控制层）
-       ⚠️ 分级上电的力矩缩放（原 `gravity_ff_scale`）现在归**控制层**的控制器参数，
-          不再是硬件 <param>。 -->
-  <xacro:arg name="gravity_ff" default="false"/>
   <xacro:arg name="joint_cfg" default="$(find motor_driver)/config/joint.yaml"/>
   <xacro:arg name="align_cfg" default="$(find arm_description)/config/align.yaml"/>
-  <xacro:arg name="mit_gains_cfg" default="$(find arm_description)/config/mit_gains.yaml"/>
   <xacro:property name="arm_cfg" value="${xacro.load_yaml('$(arg joint_cfg)')}"/>
   <xacro:property name="align_cfg" value="${xacro.load_yaml('$(arg align_cfg)')}"/>
-  <xacro:property name="mit_cfg" value="${xacro.load_yaml('$(arg mit_gains_cfg)')}"/>
   <!-- mock 的一个关节：起始姿态用 initial（模型坐标） -->
   <xacro:macro name="mock_joint" params="name initial">
     <joint name="${name}">
       <command_interface name="position"/>
-      <!-- velocity / effort 命令接口：真机插件两条链都导出（见 dm_system_interface），
-           mock 分支必须**声明同一套**，否则两条链的接口集不一致、控制器配置没法共用。 -->
-      <command_interface name="velocity"/>
+      <!-- effort 命令接口（**空插槽**）：真机插件导出它但从不读；mock 分支声明同一套，
+           否则两条链的接口集不一致、控制器配置没法共用。 -->
       <command_interface name="effort"/>
       <state_interface name="position"><param name="initial_value">${initial}</param></state_interface>
@@ -45,17 +37,11 @@
     </joint>
   </xacro:macro>
-  <!-- 真机的一个关节：参数全部从上面三个 yaml 里取 -->
+  <!-- 真机的一个关节：参数全部从上面两个 yaml 里取 -->
   <xacro:macro name="real_joint" params="name">
     <xacro:property name="jcfg" value="${arm_cfg['joints'][name]}"/>
     <xacro:property name="acfg" value="${align_cfg['joints'][name]}"/>
-    <xacro:property name="mcfg" value="${mit_cfg['joints'][name]}"/>
     <joint name="${name}">
       <command_interface name="position"/>
-      <!-- velocity 命令接口：MIT 路径把它当 `dq_des`（轨迹的 dq 从这里进来）；
-           POS_VEL 路径不看它。 -->
-      <command_interface name="velocity"/>
-      <!-- effort 命令接口：**本层选控制模式的唯一依据**（D-L1）。
-           控制器写进来的值被当作 MIT 的 `tau_ff`（前馈量）；PD 仍由硬件用下面的
-           kp_hold/kd_hold 叠加（D-L2）。没人写 ⇒ NaN ⇒ 走 POS_VEL。 -->
+      <!-- effort 命令接口：**空插槽**（见文件头）。本层永远不读它。 -->
       <command_interface name="effort"/>
       <state_interface name="position"/>     <!-- 真值从硬件读，不给 initial_value -->
@@ -76,9 +62,4 @@
       <param name="sign">${acfg['sign']}</param>
       <param name="zero_shift">${acfg['zero_shift']}</param>
-      <!-- 物理力矩上限（关节侧额定值：j1~j3 12.0 / j4~j6 3.5；与上面档位里的 t_max
-           = 电机峰值 28/10 不是一回事）+ MIT 的保持增益（D-L2：**留在硬件层**）。 -->
-      <param name="torque_max">${jcfg['torque_max']}</param>
-      <param name="kp_hold">${mcfg['kp_hold']}</param>
-      <param name="kd_hold">${mcfg['kd_hold']}</param>
     </joint>
   </xacro:macro>
@@ -97,8 +78,4 @@
           <param name="enable_on_activate">$(arg enable_on_activate)</param>
           <param name="vlim">$(arg vlim)</param>
-          <!-- 预置模式（没有控制器时发哪一种帧）：true ⇒ MIT + effort=0 / false ⇒ POS_VEL。
-               ⚠️ **不是**整链开关：真正的模式由 effort 接口每周期决定（D-L1）。
-               重力/摩擦/积分的前馈量由控制层经 effort 命令接口送来，硬件不自己算。 -->
-          <param name="gravity_ff">$(arg gravity_ff)</param>
         </hardware>
       </xacro:unless>
